File: hardware/KungFuFlash2_clean.kicad_pcb (KiCad board)
At the start: 2 copper layers, 60.6 x 62 mm, 57 parts, among them J1 DNP, J2 USB_C_Receptacle_USB2.0, J3 DNP, Q1 BC817-40, SW1 ES411X-10XX-43X-16-B, SW2 ES411X-10XX-43X-16-B, SW3 ES411X-10XX-43X-16-B, U1 Edge Connector, Immersion gol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, U2 AMS1117-3.3, U3 STM32H7B0VBTx, Y1 25 MHz

Commit message: Save KiCad panel project files
Parts:
- moved R5 2.68 mm to (109.2, 76.5)
- moved REF** 2.30 mm to (81.0, 81.9)
- moved C17 1.86 mm to (88.9, 84.0), turned to 180 degrees
- moved C16 1.85 mm to (112.6, 80.1)
- moved C9 1.00 mm to (123.7, 72.9)
- moved SW1 0.99 mm to (127.9, 73.1)
- moved SW3 0.32 mm to (82.7, 73.0)
- moved SW2 0.30 mm to (115.8, 73.0)
Routing:
- net GND: track 578.8 -> 640.0 mm
- net /MENU: track 18.1 -> 22.9 mm
- net Net-(R5-Pad1): track 6.97 -> 8.14 mm
Other:
- outline, holes or cut-outs redrawn
