File: hardware/KungFuFlash2.kicad_pcb (KiCad board)
At the start: 2 copper layers, 60.6 x 62 mm, 57 parts, among them J1 DNP, J2 USB_C_Receptacle_USB2.0, J3 DNP, Q1 BC817-40, SW1 ES411X-10XX-43X-16-B, SW2 ES411X-10XX-43X-16-B, SW3 ES411X-10XX-43X-16-B, U1 Edge Connector, Immersion gol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, U2 AMS1117-3.3, U3 STM32H7B0VBTx, Y1 25 MHz

Commit message: Update PCB layout and add connector footprint
Parts:
- moved C13 37.8 mm to (158.8, 85.7)
- moved C3 37.8 mm to (129.4, 100.3)
- moved C1 37.8 mm to (116.5, 99.8)
- moved C14 37.8 mm to (139.9, 86.4)
- moved C16 37.8 mm to (148.2, 74.6)
- moved C17 37.8 mm to (127.4, 77.0)
- moved C6 37.8 mm to (159.4, 96.1)
- moved D1 37.8 mm to (164.3, 74.7)
- moved D2 37.8 mm to (117.1, 107.5)
- moved J1 37.8 mm to (166.7, 89.8)
- moved J3 37.8 mm to (158.8, 81.5)
- moved Q1 37.8 mm to (120.7, 110.2)
- moved R10 37.8 mm to (162.3, 109.9)
- moved R12 37.8 mm to (158.1, 109.9)
- moved R16 37.8 mm to (168.9, 74.5)
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Other:
- board text added: "MANUFACTURED BY TINKERFAB Pula, Croatia Prototype · Small-Series EMS SMT · THT · Testing · Programming 0201 · 0.4 mm pitch · BGA Pilot Batch · 2026"
